Commit message: one bug but saving for safe side

File: my_arm.urdf (robot description, URDF)
Before this commit: robot simple_arm, 8 links, 7 joints
Joints:
- joint left_finger_joint: limit lower=0.0 upper=0.015 effort=1 velocity=0.1 -> lower=0.0 upper=1.5708 effort=1 velocity=0.5; type prismatic -> revolute
- joint right_finger_joint: limit lower=0.0 upper=0.015 effort=1 velocity=0.1 -> lower=0.0 upper=1.5708 effort=1 velocity=0.5

Commit message: Visual bug is fixed of rviz

File: my_arm.urdf (robot description, URDF)
Before this commit: robot simple_arm, 8 links, 7 joints
Joints:
- joint left_finger_joint: limit lower=0.0 upper=1.5708 effort=1 velocity=0.5 -> lower=0.0 upper=0.02 effort=1 velocity=0.05; type revolute -> prismatic
- joint right_finger_joint: limit lower=0.0 upper=1.5708 effort=1 velocity=0.5 -> lower=0.0 upper=0.02 effort=1 velocity=0.05

Commit message: Successfull version of urdf file v1.0.4

File: my_arm.urdf (robot description, URDF)
Before this commit: robot simple_arm, 8 links, 7 joints
Joints:
- joint right_finger_joint: mimic joint=left_finger_joint -> joint=left_finger_joint multiplier=1.0
